Commit message: feat(sim): implement Gazebo Harmonic simulation, Mecanum physics, and shared multi-terminal container
- Add MecanumDrive plugin, wheel friction tuning, and sensor plugins (LiDAR, RealSense, IMU) to robot.urdf.xacro
- Add indoor obstacle world default.sdf and ros_gz_bridge.yaml topic mappings (with /unilidar/cloud PointCloud2 and /scan LaserScan)
- Implement intel_sys_sim launch files and master sim.launch.py coordinator
- Add dead-reckoned JointState publishing in mecanum_controller.py for hardware wheel state visualization
- Keep robot_description.launch.py pure to robot_state_publisher
- Configure multi-terminal shared container in docker-compose.yml and run_docker.sh with auto bashrc sourcing
- Update Dockerfile with ros-humble-ros-gz and update README.md documentation

File: src/intel_sys_description/urdf/robot.urdf.xacro (robot description, xacro)
@@ -241,3 +241,160 @@
     <child link="camera_color_frame"/>
   </joint>
+  <!-- ==================== GAZEBO SIMULATION PLUGINS ==================== -->
+  <gazebo>
+    <!-- Mecanum Drive Plugin -->
+    <plugin filename="gz-sim-mecanum-drive-system" name="gz::sim::systems::MecanumDrive">
+      <front_left_joint>wheel_left_front_joint</front_left_joint>
+      <front_right_joint>wheel_right_front_joint</front_right_joint>
+      <back_left_joint>wheel_left_back_joint</back_left_joint>
+      <back_right_joint>wheel_right_back_joint</back_right_joint>
+      <wheel_separation>0.195</wheel_separation>
+      <wheel_base>0.216</wheel_base>
+      <wheel_radius>0.049</wheel_radius>
+      <min_velocity>-1.5</min_velocity>
+      <max_velocity>1.5</max_velocity>
+      <min_acceleration>-3.0</min_acceleration>
+      <max_acceleration>3.0</max_acceleration>
+      <topic>/cmd_vel</topic>
+      <odom_topic>/odom</odom_topic>
+      <tf_topic>/tf</tf_topic>
+      <frame_id>odom</frame_id>
+      <child_frame_id>base_footprint</child_frame_id>
+      <odom_publish_frequency>50</odom_publish_frequency>
+    </plugin>
+    <!-- Joint State Publisher for Simulated Joints -->
+    <plugin filename="gz-sim-joint-state-publisher-system" name="gz::sim::systems::JointStatePublisher">
+      <topic>/joint_states</topic>
+    </plugin>
+  </gazebo>
+  <!-- Wheel Surface Friction Workaround -->
+  <gazebo reference="wheel_right_front_link">
+    <collision>
+      <surface>
+        <friction>
+          <ode>
+            <mu>0.1</mu>
+            <mu2>0.1</mu2>
+          </ode>
+        </friction>
+      </surface>
+    </collision>
+  </gazebo>
+  <gazebo reference="wheel_left_front_link">
+    <collision>
+      <surface>
+        <friction>
+          <ode>
+            <mu>0.1</mu>
+            <mu2>0.1</mu2>
+          </ode>
+        </friction>
+      </surface>
+    </collision>
+  </gazebo>
+  <gazebo reference="wheel_right_back_link">
+    <collision>
+      <surface>
+        <friction>
+          <ode>
+            <mu>0.1</mu>
+            <mu2>0.1</mu2>
+          </ode>
+        </friction>
+      </surface>
+    </collision>
+  </gazebo>
+  <gazebo reference="wheel_left_back_link">
+    <collision>
+      <surface>
+        <friction>
+          <ode>
+            <mu>0.1</mu>
+            <mu2>0.1</mu2>
+          </ode>
+        </friction>
+      </surface>
+    </collision>
+  </gazebo>
+  <!-- Unitree L2 3D LiDAR Sensor -->
+  <gazebo reference="lidar_link">
+    <sensor name="gpu_lidar" type="gpu_lidar">
+      <always_on>true</always_on>
+      <update_rate>10</update_rate>
+      <pose relative_to="lidar_link">0 0 0 0 0 0</pose>
+      <topic>/unilidar/cloud</topic>
+      <gz_frame_id>lidar_link</gz_frame_id>
+      <lidar>
+        <scan>
+          <horizontal>
+            <samples>360</samples>
+            <resolution>1</resolution>
+            <min_angle>-3.14159265</min_angle>
+            <max_angle>3.14159265</max_angle>
+          </horizontal>
+          <vertical>
+            <samples>16</samples>
+            <resolution>1</resolution>
+            <min_angle>-0.314</min_angle>
+            <max_angle>0.314</max_angle>
+          </vertical>
+        </scan>
+        <range>
+          <min>0.1</min>
+          <max>25.0</max>
+          <resolution>0.01</resolution>
+        </range>
+      </lidar>
+    </sensor>
+  </gazebo>
+  <!-- Intel RealSense Depth Camera Sensor -->
+  <gazebo reference="camera_link">
+    <sensor name="rgbd_camera" type="rgbd_camera">
+      <always_on>true</always_on>
+      <update_rate>30</update_rate>
+      <pose relative_to="camera_link">0 0 0 0 0 0</pose>
+      <topic>/camera</topic>
+      <gz_frame_id>camera_color_frame</gz_frame_id>
+      <camera>
+        <horizontal_fov>1.5184</horizontal_fov>
+        <image>
+          <width>640</width>
+          <height>480</height>
+          <format>R8G8B8</format>
+        </image>
+        <clip>
+          <near>0.1</near>
+          <far>10.0</far>
+        </clip>
+        <depth_camera>
+          <clip>
+            <near>0.1</near>
+            <far>10.0</far>
+          </clip>
+        </depth_camera>
+      </camera>
+    </sensor>
+  </gazebo>
+  <!-- STM32 IMU Sensor -->
+  <gazebo reference="imu_link">
+    <sensor name="imu_sensor" type="imu">
+      <always_on>true</always_on>
+      <update_rate>100</update_rate>
+      <pose relative_to="imu_link">0 0 0 0 0 0</pose>
+      <topic>/imu_raw</topic>
+      <gz_frame_id>imu_link</gz_frame_id>
+      <imu>
+        <angular_velocity>
+          <x><noise type="gaussian"><mean>0.0</mean><stddev>0.0002</stddev></noise></x>
+          <y><noise type="gaussian"><mean>0.0</mean><stddev>0.0002</stddev></noise></y>
+          <z><noise type="gaussian"><mean>0.0</mean><stddev>0.0002</stddev></noise></z>
+        </angular_velocity>
+        <linear_acceleration>
+          <x><noise type="gaussian"><mean>0.0</mean><stddev>0.01</stddev></noise></x>
+          <y><noise type="gaussian"><mean>0.0</mean><stddev>0.01</stddev></noise></y>
+          <z><noise type="gaussian"><mean>0.0</mean><stddev>0.01</stddev></noise></z>
+        </linear_acceleration>
+      </imu>
+    </sensor>
+  </gazebo>
 </robot>

Commit message: feat(foxglove): refine Foxglove telemetry, docker networking, and teleop kinematics
- Expose port 8765 in docker-compose.yml for seamless Windows host WebSocket connection
- Guard docker/entrypoint.sh against recursive subshell forks when sourced in interactive shells
- Enhance run_docker.sh with TTY detection for instant interactive shell attachment
- Update robot.urdf.xacro wheel joint rotational axes to align forward/turn teleop commands with Gazebo physics
- Configure foxglove_layout.json with Z-up mesh orientation, base_link display frame, hidden TF axes by default, and color RGB camera feed
- Standardize RealSense camera launch remappings to /camera/image_raw

File: src/intel_sys_description/urdf/robot.urdf.xacro (robot description, xacro)
@@ -103,5 +103,5 @@
     <parent link="base_link"/>
     <child link="wheel_right_front_link"/>
-    <axis xyz="0 0 1"/>
+    <axis xyz="0 0 -1"/>
   </joint>
   <!-- Front Left Wheel -->
@@ -126,5 +126,5 @@
     <parent link="base_link"/>
     <child link="wheel_left_front_link"/>
-    <axis xyz="0 0 1"/>
+    <axis xyz="0 0 -1"/>
   </joint>
   <!-- Back Right Wheel -->
@@ -149,5 +149,5 @@
     <parent link="base_link"/>
     <child link="wheel_right_back_link"/>
-    <axis xyz="0 0 1"/>
+    <axis xyz="0 0 -1"/>
   </joint>
   <!-- Back Left Wheel -->
@@ -172,5 +172,5 @@
     <parent link="base_link"/>
     <child link="wheel_left_back_link"/>
-    <axis xyz="0 0 1"/>
+    <axis xyz="0 0 -1"/>
   </joint>
   <!-- ==================== SENSORS ==================== -->

Commit message: reoriented unilidar in urdf and added alias to lidar_link

File: src/intel_sys_description/urdf/robot.urdf.xacro (robot description, xacro)
@@ -198,7 +198,20 @@
   </link>
   <joint name="lidar_joint" type="fixed">
-    <origin xyz="0.0959 0.0 0.1284" rpy="0 0 0"/>
+    <origin xyz="0.0959 0.0 0.1284" rpy="0 1.5708 0"/>
     <parent link="base_link"/>
     <child link="lidar_link"/>
+  </joint>
+  <!-- Unitree Driver Hardware Frame Aliases (connects vendor frames to standard ROS tree) -->
+  <link name="unilidar_lidar"/>
+  <joint name="unilidar_lidar_alias_joint" type="fixed">
+    <origin xyz="0 0 0" rpy="0 0 0"/>
+    <parent link="lidar_link"/>
+    <child link="unilidar_lidar"/>
+  </joint>
+  <link name="unilidar_imu"/>
+  <joint name="unilidar_imu_alias_joint" type="fixed">
+    <origin xyz="0 0 0" rpy="0 0 0"/>
+    <parent link="lidar_link"/>
+    <child link="unilidar_imu"/>
   </joint>
   <!-- Intel RealSense Depth Camera -->

Commit message: fixed unitree frame issues

File: src/intel_sys_description/urdf/robot.urdf.xacro (robot description, xacro)
@@ -198,20 +198,14 @@
   </link>
   <joint name="lidar_joint" type="fixed">
-    <origin xyz="0.0959 0.0 0.1284" rpy="0 1.5708 0"/>
+    <origin xyz="0.0959 0.0 0.1284" rpy="0 ${-pi/2} ${pi}"/>
     <parent link="base_link"/>
     <child link="lidar_link"/>
   </joint>
-  <!-- Unitree Driver Hardware Frame Aliases (connects vendor frames to standard ROS tree) -->
-  <link name="unilidar_lidar"/>
-  <joint name="unilidar_lidar_alias_joint" type="fixed">
-    <origin xyz="0 0 0" rpy="0 0 0"/>
+  <!-- Unitree L2 Internal IMU -->
+  <link name="lidar_imu_link"/>
+  <joint name="lidar_imu_joint" type="fixed">
+    <origin xyz="0.007698 0.014655 -0.00667" rpy="0 0 0"/>
     <parent link="lidar_link"/>
-    <child link="unilidar_lidar"/>
-  </joint>
-  <link name="unilidar_imu"/>
-  <joint name="unilidar_imu_alias_joint" type="fixed">
-    <origin xyz="0 0 0" rpy="0 0 0"/>
-    <parent link="lidar_link"/>
-    <child link="unilidar_imu"/>
+    <child link="lidar_imu_link"/>
   </joint>
   <!-- Intel RealSense Depth Camera -->
@@ -370,5 +364,5 @@
       <pose relative_to="lidar_link">0.007698 0.014655 -0.00667 0 0 0</pose>
       <topic>/lidar/imu</topic>
-      <gz_frame_id>lidar_link</gz_frame_id>
+      <gz_frame_id>lidar_imu_link</gz_frame_id>
       <imu>
         <angular_velocity>
